File: P1/pcb/alu_addsub/alu.kicad_pcb (KiCad board)
At the start: 4 copper layers, 100.3 x 100.3 mm, 35 parts, among them J1 650473-5, U1 74HC86, U10 74LS08, U13 74LS541, U14 74HC86, U15 74HC86, U2 74LS08, U29 74HC238, U3 74LS32, U30 74LS32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

Commit message: Removed unneeded backup files
Connections:
- J1 pad A18: /X_IN0 -> GND
- J1 pad A19: /X_IN1 -> /X_IN0
- J1 pad A20: /X_IN2 -> /X_IN1
- J1 pad A21: /X_IN3 -> /X_IN2
- J1 pad A22: /X_IN4 -> /X_IN3
- J1 pad A23: /X_IN5 -> /X_IN4
- J1 pad A24: /X_IN6 -> /X_IN5
- J1 pad A25: /X_IN7 -> /X_IN6
- J1 pad A26: unconnected-(J1-PadA26) -> /X_IN7
Routing:
- net /X_IN7: track 38.1 -> 32.7 mm
- net /X_IN5: track 40.5 -> 35.4 mm
- net /X_IN6: track 38.7 -> 34.0 mm
- net /X_IN2: track 42.5 -> 39.3 mm
- net /X_IN4: track 40.4 -> 37.6 mm
- net /X_IN3: track 41.6 -> 38.9 mm
- net /X_IN1: track 43.2 -> 40.7 mm
- net /X_IN0: track 44.2 -> 42.4 mm
