File: P1/pcb/alu_binary_op/alu.kicad_pcb (KiCad board)
At the start: 4 copper layers, 100.3 x 100.3 mm, 25 parts, among them J1 650473-5, U13 74LS541, U14 74HC86, U15 74HC86, U16 74LS621, U17 74LS08, U18 74LS08, U19 74LS621, U20 74LS32, U21 74LS32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

Commit message: Removed unneeded backup files
Connections:
- J1 pad A18: /X_IN0 -> GND
- J1 pad A19: /X_IN1 -> /X_IN0
- J1 pad A20: /X_IN2 -> /X_IN1
- J1 pad A21: /X_IN3 -> /X_IN2
- J1 pad A22: /X_IN4 -> /X_IN3
- J1 pad A23: /X_IN5 -> /X_IN4
- J1 pad A24: /X_IN6 -> /X_IN5
- J1 pad A25: /X_IN7 -> /X_IN6
- J1 pad A26: unconnected-(J1-PadA26) -> /X_IN7
Routing:
- net GND: track 196.0 -> 202.1 mm
- net /X_IN5: track 82.9 -> 85.1 mm
- net /X_IN1: track 78.7 -> 77.5 mm
- net /X_IN6: track 85.5 -> 86.5 mm
- net /X_IN3: track 80.3 -> 81.2 mm
- net /X_IN4: track 82.8 -> 82.3 mm
