File: P1/pcb/alu_unary_op/alu.kicad_sch (KiCad schematic)
At the start: 19 parts, among them J1 650473-5, U13 74LS541, U23 74HC04, U24 74HC04, U25 74LS621, U26 74LS157, U27 74LS157, U28 74LS621, U29 74HC238, U30 74LS32

Commit message: Removed unneeded backup files
Connections:
- net GND: now also J1.A18
- net X_IN0: now also J1.A19; no longer J1.A18
- net X_IN1: now also J1.A20; no longer J1.A19
- net X_IN2: now also J1.A21; no longer J1.A20
- net X_IN3: now also J1.A22; no longer J1.A21
- net X_IN4: now also J1.A23; no longer J1.A22
- net X_IN5: now also J1.A24; no longer J1.A23
- net X_IN6: now also J1.A25; no longer J1.A24
- net X_IN7: now also J1.A26; no longer J1.A25
Changed lines of the file:
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@@
 	)
 	(junction
+		(at 119.38 73.66)
+		(diameter 0)
+		(color 0 0 0 0)
+	)
+	(junction
 		(at 1167.13 39.37)
 		(diameter 0)
@@
 	)
 	(bus_entry
-		(at 123.19 73.66)
-		(size 2.54 -2.54)
-		(stroke
-			(width 0)
-			(type default)
-		)
-	)
-	(bus_entry
 		(at 120.65 336.55)
 		(size 2.54 2.54)
@@
 	(wire
 		(pts
+			(xy 119.38 73.66) (xy 119.38 90.17)
+		)
+		(stroke
+			(width 0)
+			(type default)
+		)
+	)
+	(wire
+		(pts
 			(xy 190.5 359.41) (xy 205.74 359.41)
 		)
@@
 	(wire
 		(pts
+			(xy 110.49 73.66) (xy 119.38 73.66)
+		)
+		(stroke
+			(width 0)
+			(type default)
+		)
+	)
+	(wire
+		(pts
 			(xy 303.53 212.09) (xy 303.53 218.44)
 		)
@@
 		)
 	)
-	(bus
-		(pts
-			(xy 125.73 68.58) (xy 125.73 71.12)
-		)
-		(stroke
-			(width 0)
-			(type default)
-		)
-	)
 	(wire
 		(pts
@@
 	(wire
 		(pts
-			(xy 110.49 73.66) (xy 123.19 73.66)
-		)
-		(stroke
-			(width 0)
-			(type default)
-		)
-	)
-	(wire
-		(pts
 			(xy 264.16 292.1) (xy 264.16 274.32)
 		)
@@
 	(wire
 		(pts
-			(xy 119.38 50.8) (xy 119.38 90.17)
+			(xy 119.38 50.8) (xy 119.38 73.66)
 		)
 		(stroke
@@
 	(bus
 		(pts
-			(xy 125.73 71.12) (xy 125.73 92.71)
+			(xy 125.73 68.58) (xy 125.73 92.71)
 		)
 		(stroke
@@
 		)
 	)
-	(label "X_IN6"
-		(at 111.76 58.42 0)
-		(fields_autoplaced yes)
-		(effects
-			(font
-				(size 1.27 1.27)
-			)
-			(justify left bottom)
-		)
-	)
 	(label "X_IN1"
 		(at 344.17 370.84 0)
@@
 		)
 	)
-	(label "X_OUT3"
-		(at 83.82 180.34 0)
+	(label "X_IN2"
+		(at 111.76 66.04 0)
 		(fields_autoplaced yes)
 		(effects
@@
 		)
 	)
-	(label "X_IN7"
-		(at 111.76 55.88 0)
+	(label "X_OUT3"
+		(at 83.82 180.34 0)
 		(fields_autoplaced yes)
 		(effects
@@
 		)
 	)
-	(label "X_IN0"
-		(at 111.76 73.66 0)
-		(fields_autoplaced yes)
-		(effects
-			(font
-				(size 1.27 1.27)
-			)
-			(justify left bottom)
-		)
-	)
 	(label "X_OUT7"
 		(at 127 427.99 0)
@@
 		)
 	)
+	(label "X_IN4"
+		(at 111.76 60.96 0)
+		(fields_autoplaced yes)
+		(effects
+			(font
+				(size 1.27 1.27)
+			)
+			(justify left bottom)
+		)
+	)
 	(label "X_IN7"
 		(at 344.17 279.4 0)
@@
 		)
 	)
-	(label "X_IN5"
-		(at 111.76 60.96 0)
+	(label "X_OUT4"
+		(at 83.82 177.8 0)
 		(fields_autoplaced yes)
 		(effects
@@
 		)
 	)
-	(label "X_OUT4"
-		(at 83.82 177.8 0)
+	(label "X_IN6"
+		(at 111.76 55.88 0)
 		(fields_autoplaced yes)
 		(effects
@@
 		)
 	)
-	(label "X_IN4"
-		(at 111.76 63.5 0)
-		(fields_autoplaced yes)
-		(effects
-			(font
-				(size 1.27 1.27)
-			)
-			(justify left bottom)
-		)
-	)
 	(label "X_OUT5"
 		(at 127 276.86 0)
@@
 		)
 	)
-	(label "X_IN3"
-		(at 111.76 66.04 0)
+	(label "X_IN5"
+		(at 111.76 58.42 0)
 		(fields_autoplaced yes)
 		(effects
@@
 		)
 	)
-	(label "X_IN1"
-		(at 111.76 71.12 0)
+	(label "X_IN7"
+		(at 111.76 53.34 0)
 		(fields_autoplaced yes)
 		(effects
@@
 		)
 	)
-	(label "X_IN2"
-		(at 111.76 68.58 0)
+	(label "X_IN1"
+		(at 344.17 248.92 0)
 		(fields_autoplaced yes)
 		(effects
@@
 		)
 	)
-	(label "X_IN1"
-		(at 344.17 248.92 0)
+	(label "X_OUT5"
+		(at 127 397.51 0)
 		(fields_autoplaced yes)
 		(effects
@@
 		)
 	)
-	(label "X_OUT5"
-		(at 127 397.51 0)
+	(label "X_IN1"
+		(at 111.76 68.58 0)
 		(fields_autoplaced yes)
 		(effects
@@
 		)
 	)
+	(label "X_IN3"
+		(at 111.76 63.5 0)
+		(fields_autoplaced yes)
+		(effects
+			(font
+				(size 1.27 1.27)
+			)
+			(justify left bottom)
+		)
+	)
 	(label "X_OUT0"
 		(at 125.73 322.58 0)
@@
 		(fields_autoplaced yes)
 		(effects
+			(font
+				(size 1.27 1.27)
+			)
+			(justify left bottom)
+		)
+	)
+	(label "X_IN0"
+		(at 111.76 71.12 0)
+		(fields_autoplaced yes)
+		(effects
