File: P1/pcb/the_stack/the_stack.kicad_sch (KiCad schematic)
At the start: 44 parts, among them J1 650473-5, U1 X_0, U10 74LS157, U11 74LS157, U12 74LS157, U13 74LS157, U14 74LS157, U15 74LS621, U16 74LS157, U17 74LS157, U18 74HCT238, U19 74LS32, U2 X, U20 74LS32, U21 74LS14, U22 74LS14, U23 74LS08, U24 74LS08, U3 Y, U4 Z, U5 T, U6 74AHC541, U7 74AHC541, U8 74LS621, U9 74LS157

Commit message: Removed unneeded backup files
Parts:
- removed U15: 74LS621, symbol 74xx_IEEE:74LS621
- added C20, C21, C22, C23, C24, C25: 100n, symbol Device:C_Small
Connections:
- net +5V: now also U16.16 (VCC), U17.16 (VCC), U19.14 (VCC), U20.14 (VCC), U21.14 (VCC), U21.5, U22.11, U22.13, U22.14 (VCC), U23.14 (VCC), U24.14 (VCC), C20.1, C21.1, C22.1, C23.1, C24.1, C25.1
- net GND: now also U16.15 (E), U16.8 (GND), U17.15 (E), U17.8 (GND), U19.7 (GND), U20.7 (GND), U21.7 (GND), U22.7 (GND), U23.7 (GND), U24.10, U24.12, U24.13, U24.4, U24.5, U24.7 (GND), U24.9, C20.2, C21.2, C22.2, C23.2, C24.2, C25.2
- no-connect marks 47 -> 53
Other:
- moved on the sheet: U19E, U20E, U21C, U21G, U22E, U22F, U22G, U23E, U24B, U24C, U24D, U24E
